File: PCB_Main.kicad_pcb (KiCad board)
At the start: 2 copper layers, 101.6 x 53.3 mm, 38 parts, among them J1 Power, J2 PWM, J3 Analog, J4 PWM, J5 Analog, J6 Communication, J7 Conn_01x03, J8 Conn_01x03, M78AR05-1 M78AR05, M78AR05-2 M78AR05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

Commit message: update
Parts:
- removed J7, J8: Conn_01x03, Connector_PinSocket_2.54mm:PinSocket_1x03_P2.54mm_Vertical
- removed LED3: Air, LED_THT:LED_D3.0mm_Clear
- removed LED4: Under, LED_THT:LED_D3.0mm_Clear
- removed LED5: Power, LED_THT:LED_D3.0mm_Clear
- removed LED6: 1PPS, LED_THT:LED_D3.0mm_Clear
- added U1: MOUDLE-SEEEDUINO-XIAO, XIAO_PCB:MOUDLE14P-2.54-21X17.8MM, F.Cu at (113.0, 61.0)
- AE-MICRO-SD-DIP1, M78AR05-1: moved to B.Cu
- GPS-UART1: value GPS-UART -> GPS-TWE-UART
- LED1: value SD -> Conn_01x04_Female; footprint LED_THT:LED_D3.0mm_Clear -> Connector_JST:JST_XH_S4B-XH-A_1x04_P2.50mm_Horizontal
- LED2: value ICS -> Conn_01x04_Female; footprint LED_THT:LED_D3.0mm_Clear -> Connector_JST:JST_XH_S4B-XH-A_1x04_P2.50mm_Horizontal
- moved Speaker1 97.3 mm to (93.4, 75.9), turned to -90 degrees
- moved LED2 86.8 mm to (189.2, 78.7), turned to 90 degrees
- moved AE-MICRO-SD-DIP1 81.5 mm to (102.4, 59.7), turned to 90 degrees
- moved C1 76.8 mm to (120.0, 77.5), turned to -90 degrees
- moved ICS-UART1 36.8 mm to (93.4, 87.1)
- moved M78AR05-1 36.7 mm to (96.5, 86.4)
- moved Air-UART1 33.4 mm to (93.3, 55.9)
- moved Under-UART1 21.2 mm to (101.7, 90.2), turned to 0 degrees
- moved M78AR05-3 12.8 mm to (104.7, 81.2), turned to 90 degrees
- moved GPS-UART1 11.1 mm to (189.3, 64.7)
- moved LED1 9.91 mm to (189.2, 92.7), turned to 90 degrees
- moved M78AR05-2 7.59 mm to (110.1, 76.2)
- moved G*** 7.00 mm to (177.8, 77.1)
Connections:
- AE-MICRO-SD-DIP1 pad 4: 3.3V -> RP3.3V
- ATP3012 pad 15: Net-(ATP3012-Pad15) -> unconnected-(ATP3012-Pad15)
- J2 pad 5: L_ICS -> /*13
- J2 pad 6: L_Under -> /*12
- J3 pad 1: L_Air -> /A0
- J4 pad 7: /TX0/1 -> DTAR
- J4 pad 8: IRXT -> DRAT
- J5 pad 1: SD-CS -> /A8
- J5 pad 4: L_SD -> L_Air
- J5 pad 5: /A12 -> L_Under
- J5 pad 6: /A13 -> L_ICS
- J6 pad 1: DTUR -> DTSR
- J6 pad 2: DRUT -> IRXT
- J6 pad 3: DTAR -> DTUR
- J6 pad 4: DRAT -> DRUT
- LED1 pad 2: L_SD -> L_ICS
- LED2 pad 2: L_ICS -> unconnected-(LED2-Pad2)
- Speaker1 pad 3: Net-(ATP3012-Pad15) -> unconnected-(Speaker1-Pad3)
Routing:
- net GND: track 454.3 -> 324.0 mm
- net 5V: track 98.7 -> 200.0 mm
- net DTSR: track 0.00 -> 61.2 mm
- net IRXT: track 87.7 -> 121.8 mm
- net L_Under: track 44.1 -> 12.1 mm
- net L_Air: track 45.1 -> 15.6 mm
- net EN: track 33.4 -> 61.9 mm
- net 1PPS: track 0.00 -> 23.6 mm
- net ITXR: track 40.6 -> 63.5 mm
- net Net-(ATP3012-Pad15): track 21.2 -> 0.00 mm
- net RP3.3V: track 0.00 -> 20.6 mm
- net SD-CS: track 24.6 -> 5.32 mm
- net DTAR: track 91.8 -> 72.6 mm
- net Net-(Air-UART1-Pad2): track 7.97 -> 26.9 mm
- net SDA: track 123.0 -> 105.1 mm
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Other:
- board size 101.6 x 53.3 mm -> 118 x 53.3 mm

Commit message: update
Parts:
- added D1: D, Diode_THT:D_A-405_P12.70mm_Horizontal, F.Cu at (120.0, 59.1)
- added D2: D, Diode_THT:D_A-405_P10.16mm_Horizontal, F.Cu at (94.7, 74.3)
- added D3: D, Diode_THT:D_A-405_P10.16mm_Horizontal, F.Cu at (82.3, 74.3)
- added D4: D, Diode_THT:D_A-405_P10.16mm_Horizontal, F.Cu at (107.2, 74.3)
- added ICS-SW1: SW_DPDT_x2, Connector_PinHeader_2.54mm:PinHeader_1x03_P2.54mm_Vertical, B.Cu at (73.3, 86.4)
- added Serial-SW1: SW_DPDT_x2, Button_Switch_THT:SW_Push_2P2T_Toggle_CK_PVA2OAH5xxxxxxV2, B.Cu at (73.4, 81.0)
- M78AR05-1: moved to F.Cu
- U1: value MOUDLE-SEEEDUINO-XIAO -> SEEEDUINO-XIAO
- moved Speaker1 24.6 mm to (73.3, 90.1), turned to 0 degrees
- moved M78AR05-3 19.0 mm to (86.2, 76.8), turned to -90 degrees
- moved Air-UART1 13.7 mm to (79.7, 55.9)
- moved AE-MICRO-SD-DIP1 12.7 mm to (89.7, 59.7)
- moved U1 11.4 mm to (101.6, 61.0)
- moved M78AR05-1 9.77 mm to (98.7, 76.8)
- moved ICS-UART1 8.95 mm to (85.0, 90.1), turned to 0 degrees
- moved M78AR05-2 1.19 mm to (111.1, 76.8)
- moved C1 1.02 mm to (121.0, 77.4)
Connections:
- J4 pad 7: DTAR -> /TX0/1
- J4 pad 8: DRAT -> /RX0/0
- J6 pad 2: IRXT -> /RX3/15
- M78AR05-1 pad 1: VCC -> Net-(M78AR05-1-Pad1)
- M78AR05-2 pad 1: VCC -> Net-(M78AR05-2-Pad1)
- M78AR05-3 pad 1: VCC -> Net-(M78AR05-3-Pad1)
- U1 pad 14: 5V -> Net-(U1-Pad14)
Routing:
- net /RX3/15: track 0.00 -> 123.5 mm
- net /TX0/1: track 0.00 -> 104.5 mm
- net /RX0/0: track 0.00 -> 98.6 mm
- net DRAT: track 76.2 -> 14.7 mm
- net DTAR: track 72.6 -> 23.8 mm
- net GND: track 324.0 -> 369.4 mm
- net IRXT: track 121.8 -> 77.5 mm
- net Net-(M78AR05-2-Pad3): track 11.4 -> 35.2 mm
- net Net-(ICS-UART1-Pad2): track 3.94 -> 17.6 mm
- net Net-(U1-Pad14): track 0.00 -> 13.2 mm
- net DTSR: track 61.2 -> 72.6 mm
- net EN: track 61.9 -> 50.5 mm
- net 5V: track 200.0 -> 194.7 mm
- net SD-MOSI: track 26.1 -> 31.3 mm
- net Net-(M78AR05-3-Pad1): track 0.00 -> 4.99 mm
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Other:
- board size 118 x 53.3 mm -> 131.9 x 53.3 mm

Commit message: jlcpcb
Parts:
- moved ICS-SW1 36.8 mm to (73.3, 49.5)
- moved Serial-SW1 16.8 mm to (73.0, 97.8)
- moved C1 11.5 mm to (119.4, 66.0), turned to 0 degrees
- moved D1 11.2 mm to (111.8, 51.4)
- moved Speaker1 10.3 mm to (78.7, 81.4), turned to -90 degrees
- moved G*** 9.98 mm to (175.3, 67.4)
- moved AE-MICRO-SD-DIP1 5.90 mm to (88.3, 65.4)
- moved Air-UART1 5.53 mm to (78.8, 61.4)
- moved D2 5.47 mm to (100.2, 74.3)
- moved D4 5.47 mm to (112.7, 74.3)
- moved M78AR05-1 5.47 mm to (104.2, 76.8)
- moved M78AR05-2 5.47 mm to (116.6, 76.8)
- moved M78AR05-3 4.97 mm to (91.2, 76.8)
- moved U1 2.34 mm to (100.3, 59.0)
- moved D3 2.16 mm to (84.5, 74.3)
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Connections:
- ATP3012 pad 15: unconnected-(ATP3012-Pad15) -> Net-(ATP3012-Pad15)
- LED2 pad 2: unconnected-(LED2-Pad2) -> L_SD
- Speaker1 pad 3: unconnected-(Speaker1-Pad3) -> Net-(ATP3012-Pad15)
- U1 pad 2: unconnected-(U1-Pad2) -> L_SD
Routing:
- net L_SD: track 0.00 -> 114.8 mm, vias 0 -> 4
- net Net-(ATP3012-Pad15): track 0.00 -> 106.1 mm
- net IRXT: track 77.5 -> 139.4 mm
- net GND: track 369.4 -> 398.8 mm
- net /RX3/15: track 123.5 -> 100.0 mm
- net 5V: track 194.7 -> 213.3 mm
- net /TX0/1: track 104.5 -> 122.6 mm
- net Net-(M78AR05-2-Pad3): track 35.2 -> 17.8 mm
- net /RX0/0: track 98.6 -> 115.9 mm
- net DTAR: track 23.8 -> 35.3 mm
- net DRAT: track 14.7 -> 26.0 mm
- net Net-(D1-Pad1): track 13.2 -> 3.84 mm
- net DTUR: track 97.4 -> 91.9 mm
- net VCC: track 72.4 -> 68.1 mm
- net DRUT: track 95.4 -> 91.5 mm
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Other:
- board text added: "3.3V 1PPS SD GND"
- board text added: "Air Under ICS GND"
- board text removed: "ICSP"
