File: PCB_Main.kicad_sch (KiCad schematic)
At the start: 30 parts, among them J1 Power, J2 PWM, J3 Analog, J4 PWM, J5 Analog, J6 Communication, J7 Conn_01x03, J8 Conn_01x03, U1 DPS310, U2 ATP3012, U3 R-78E5.0-1.0, U4 R-78E5.0-1.0, U5 R-78E5.0-1.0, U6 AE-BNO055, U7 ICS, Y1 16MHｚ

Commit message: update silk
Parts:
- 1PPS1: value LED -> 1PPS
- AE-MICRO-SD-DIP1: value Micro_SD_Card_Det_Hirose_DM3AT -> AE-MICRO-SD-DIP
- Air-UART1: value Conn_01x04_Female -> Air-UART
- Air1: value LED -> Air
- GPS-UART1: value Conn_01x05_Female -> GPS-UART
- ICS-UART1: value Conn_01x05_Female -> ICS-UART
- ICS1: value LED -> ICS
- M78AR05-1: renamed from U3; value R-78E5.0-1.0 -> M78AR05
- M78AR05-2: renamed from U5; value R-78E5.0-1.0 -> M78AR05
- M78AR05-3: renamed from U4; value R-78E5.0-1.0 -> M78AR05
- Power1: value LED -> Power
- SD1: value LED -> SD
- Speaker1: value Conn_01x03_Female -> Speaker
- Under-UART1: value Conn_01x04_Female -> Under-UART
- Under1: value LED -> Under
- renumbered U6 to AE-BNO55, U2 to ATP3012, U1 to DPS310, U7 to ICS-board1
Other:
- note removed: "* Indicates a PWM-capable pin"
- company: (none) -> TORICA-23th
- title: (none) -> Main
- moved on the sheet: 1PPS1, AE-BNO55, AE-MICRO-SD-DIP1, Air1, DPS310, ICS-board1, ICS1, Power1, SD1, Under1

Commit message: pass DRC
Parts:
- renumbered AE-BNO55 to AE-BNO055, Power1 to LED, ICS1 to LED, Air1 to LED, Under1 to LED, SD1 to LED, 1PPS1 to LED
Changed lines of the file:
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@@
   (symbol (lib_id "Device:LED") (at 76.2 161.29 90) (unit 1)
     (in_bom yes) (on_board yes) (fields_autoplaced)
-    (property "Reference" "Power1" (id 0) (at 80.01 161.6074 90)
+    (property "Reference" "LED" (id 0) (at 80.01 161.6074 90)
       (effects (font (size 1.27 1.27)) (justify right))
     )
@@
   )
   (symbol (lib_id "Connector_Generic:Conn_01x03") (at 139.7 101.6 270) (unit 1)
-    (in_bom yes) (on_board yes) (fields_autoplaced)
+    (in_bom yes) (on_board yes)
     (property "Reference" "J7" (id 0) (at 144.78 100.3299 90)
       (effects (font (size 1.27 1.27)) (justify left))
     )
-    (property "Value" "Conn_01x03" (id 1) (at 144.78 102.8699 90)
+    (property "Value" "Conn_01x03" (id 1) (at 133.35 104.14 90)
       (effects (font (size 1.27 1.27)) (justify left))
     )
@@
   (symbol (lib_id "Device:LED") (at 40.64 161.29 90) (unit 1)
     (in_bom yes) (on_board yes)
-    (property "Reference" "ICS1" (id 0) (at 44.45 161.6074 90)
+    (property "Reference" "LED" (id 0) (at 44.45 161.6074 90)
       (effects (font (size 1.27 1.27)) (justify right))
     )
@@
   (symbol (lib_id "Device:LED") (at 52.07 161.29 90) (unit 1)
     (in_bom yes) (on_board yes)
-    (property "Reference" "Air1" (id 0) (at 55.88 161.6074 90)
+    (property "Reference" "LED" (id 0) (at 55.88 161.6074 90)
       (effects (font (size 1.27 1.27)) (justify right))
     )
@@
   )
   (symbol (lib_id "Connector_Generic:Conn_01x03") (at 139.7 110.49 90) (unit 1)
-    (in_bom yes) (on_board yes) (fields_autoplaced)
+    (in_bom yes) (on_board yes)
     (property "Reference" "J8" (id 0) (at 144.78 109.2199 90)
       (effects (font (size 1.27 1.27)) (justify right))
     )
-    (property "Value" "Conn_01x03" (id 1) (at 144.78 111.7599 90)
+    (property "Value" "Conn_01x03" (id 1) (at 133.35 107.95 90)
       (effects (font (size 1.27 1.27)) (justify right))
     )
@@
   (symbol (lib_id "Device:LED") (at 63.5 161.29 90) (unit 1)
     (in_bom yes) (on_board yes) (fields_autoplaced)
-    (property "Reference" "Under1" (id 0) (at 67.31 161.6074 90)
+    (property "Reference" "LED" (id 0) (at 67.31 161.6074 90)
       (effects (font (size 1.27 1.27)) (justify right))
     )
@@
   (symbol (lib_id "AE-BNO055:AE-BNO055") (at 50.8 77.47 0) (unit 1)
     (in_bom yes) (on_board yes) (fields_autoplaced)
-    (property "Reference" "AE-BNO55" (id 0) (at 56.515 72.39 0))
+    (property "Reference" "AE-BNO055" (id 0) (at 56.515 72.39 0))
     (property "Value" "AE-BNO055" (id 1) (at 56.515 74.93 0))
     (property "Footprint" "AE-BNO055:AE-BNO055" (id 2) (at 48.26 76.2 0)
@@
   (symbol (lib_id "Device:LED") (at 29.21 161.29 90) (unit 1)
     (in_bom yes) (on_board yes)
-    (property "Reference" "SD1" (id 0) (at 33.02 161.6074 90)
+    (property "Reference" "LED" (id 0) (at 33.02 161.6074 90)
       (effects (font (size 1.27 1.27)) (justify right))
     )
@@
   (symbol (lib_id "Device:LED") (at 88.9 161.29 90) (unit 1)
     (in_bom yes) (on_board yes) (fields_autoplaced)
-    (property "Reference" "1PPS1" (id 0) (at 92.71 161.6074 90)
+    (property "Reference" "LED" (id 0) (at 92.71 161.6074 90)
       (effects (font (size 1.27 1.27)) (justify right))
     )
@@
       (reference "#PWR0125") (unit 1) (value "+3.3V") (footprint "")
     )
-    (path "/edbca3e4-fedc-4bbf-9139-3f1d974c7d83"
-      (reference "1PPS1") (unit 1) (value "1PPS") (footprint "LED_THT:LED_D3.0mm_Clear")
-    )
     (path "/d000c252-ded3-41d5-b3e4-49cb65069666"
-      (reference "AE-BNO55") (unit 1) (value "AE-BNO055") (footprint "AE-BNO055:AE-BNO055")
+      (reference "AE-BNO055") (unit 1) (value "AE-BNO055") (footprint "AE-BNO055:AE-BNO055")
     )
     (path "/e5435c51-2c5d-4ddb-9b5b-d7beb7cc7dac"
@@
       (reference "Air-UART1") (unit 1) (value "Air-UART") (footprint "Connector_JST:JST_XH_S4B-XH-A_1x04_P2.50mm_Horizontal")
     )
-    (path "/b0cf4776-0395-4863-86c7-b7801a1cac53"
-      (reference "Air1") (unit 1) (value "Air") (footprint "LED_THT:LED_D3.0mm_Clear")
-    )
     (path "/729b01ec-738f-43c5-822b-27d350075413"
       (reference "DPS310") (unit 1) (value "DPS310") (footprint "DPS310:DPS310")
@@
       (reference "ICS-board1") (unit 1) (value "ICS") (footprint "ICS:ICS")
     )
-    (path "/40dc120f-8d94-48d8-afb4-92f0e8601a29"
-      (reference "ICS1") (unit 1) (value "ICS") (footprint "LED_THT:LED_D3.0mm_Clear")
-    )
     (path "/00000000-0000-0000-0000-000056d71773"
       (reference "J1") (unit 1) (value "Power") (footprint "Connector_PinHeader_2.54mm:PinHeader_1x08_P2.54mm_Vertical")
@@
       (reference "J8") (unit 1) (value "Conn_01x03") (footprint "Connector_PinSocket_2.54mm:PinSocket_1x03_P2.54mm_Vertical")
     )
+    (path "/18fb8f6b-b9c7-4385-ba05-b65cf395b9ea"
+      (reference "LED") (unit 1) (value "Power") (footprint "LED_THT:LED_D3.0mm_Clear")
+    )
+    (path "/40dc120f-8d94-48d8-afb4-92f0e8601a29"
+      (reference "LED") (unit 1) (value "ICS") (footprint "LED_THT:LED_D3.0mm_Clear")
+    )
+    (path "/b0cf4776-0395-4863-86c7-b7801a1cac53"
+      (reference "LED") (unit 1) (value "Air") (footprint "LED_THT:LED_D3.0mm_Clear")
+    )
+    (path "/ca4f06d4-e667-4d24-afc1-294ab6c4ef73"
+      (reference "LED") (unit 1) (value "Under") (footprint "LED_THT:LED_D3.0mm_Clear")
+    )
+    (path "/e8fe42a8-ca43-40a0-808f-01a629a50f73"
+      (reference "LED") (unit 1) (value "SD") (footprint "LED_THT:LED_D3.0mm_Clear")
+    )
+    (path "/edbca3e4-fedc-4bbf-9139-3f1d974c7d83"
+      (reference "LED") (unit 1) (value "1PPS") (footprint "LED_THT:LED_D3.0mm_Clear")
+    )
     (path "/2fb9aea4-6f16-4bbe-8658-1d9caff83ec7"
       (reference "M78AR05-1") (unit 1) (value "M78AR05") (footprint "Converter_DCDC:Converter_DCDC_RECOM_R-78E-0.5_THT")
@@
       (reference "M78AR05-3") (unit 1) (value "M78AR05") (footprint "Converter_DCDC:Converter_DCDC_RECOM_R-78E-0.5_THT")
     )
-    (path "/18fb8f6b-b9c7-4385-ba05-b65cf395b9ea"
-      (reference "Power1") (unit 1) (value "Power") (footprint "LED_THT:LED_D3.0mm_Clear")
-    )
     (path "/1cb880d1-9888-498d-8327-a515280ce39c"
       (reference "R1") (unit 1) (value "2k") (footprint "Resistor_THT:R_Axial_DIN0204_L3.6mm_D1.6mm_P7.62mm_Horizontal")
@@
       (reference "R2") (unit 1) (value "2k") (footprint "Resistor_THT:R_Axial_DIN0204_L3.6mm_D1.6mm_P7.62mm_Horizontal")
     )
-    (path "/e8fe42a8-ca43-40a0-808f-01a629a50f73"
-      (reference "SD1") (unit 1) (value "SD") (footprint "LED_THT:LED_D3.0mm_Clear")
-    )
     (path "/a2733bf0-4e46-4ed0-bf6b-950d686d27fd"
       (reference "Speaker1") (unit 1) (value "Speaker") (footprint "Connector_JST:JST_XH_S3B-XH-A_1x03_P2.50mm_Horizontal")
@@
       (reference "Under-UART1") (unit 1) (value "Under-UART") (footprint "Connector_JST:JST_XH_S4B-XH-A_1x04_P2.50mm_Horizontal")
     )
-    (path "/ca4f06d4-e667-4d24-afc1-294ab6c4ef73"
-      (reference "Under1") (unit 1) (value "Under") (footprint "LED_THT:LED_D3.0mm_Clear")
-    )
     (path "/98548798-5531-49e6-8f6d-89e3d12b4624"

Commit message: add capacitor
Parts:
- added C1: C_5V, Capacitor_THT:CP_Radial_D5.0mm_P2.50mm, symbol Device:C_Polarized
- renumbered AE-BNO055 to AE-BNO55, LED to LED1, LED to LED2, LED to LED3, LED to LED4, LED to LED5, LED to LED6
Connections:
- net +5V: now also C1.1
- net GND: now also C1.2
Changed lines of the file:
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@@
   (symbol (lib_id "Device:LED") (at 76.2 161.29 90) (unit 1)
     (in_bom yes) (on_board yes) (fields_autoplaced)
-    (property "Reference" "LED" (id 0) (at 80.01 161.6074 90)
+    (property "Reference" "LED5" (id 0) (at 80.01 161.6074 90)
       (effects (font (size 1.27 1.27)) (justify right))
     )
@@
   (symbol (lib_id "Device:LED") (at 40.64 161.29 90) (unit 1)
     (in_bom yes) (on_board yes)
-    (property "Reference" "LED" (id 0) (at 44.45 161.6074 90)
+    (property "Reference" "LED2" (id 0) (at 44.45 161.6074 90)
       (effects (font (size 1.27 1.27)) (justify right))
     )
@@
     (pin "1")
     (pin "2")
+  )
+  (symbol (lib_id "power:+5V") (at 146.05 25.4 0) (unit 1)
+    (in_bom yes) (on_board yes) (fields_autoplaced)
+    (property "Reference" "#PWR0127" (id 0) (at 146.05 29.21 0)
+      (effects (font (size 1.27 1.27)) hide)
+    )
+    (property "Value" "+5V" (id 1) (at 146.05 20.32 0))
+    (property "Footprint" "" (id 2) (at 146.05 25.4 0)
+      (effects (font (size 1.27 1.27)) hide)
+    )
+    (property "Datasheet" "" (id 3) (at 146.05 25.4 0)
+      (effects (font (size 1.27 1.27)) hide)
+    )
+    (pin "1")
   )
   (symbol (lib_id "power:VCC") (at 118.11 48.26 0) (unit 1)
@@
     (pin "1")
   )
+  (symbol (lib_id "power:GND") (at 146.05 33.02 0) (unit 1)
+    (in_bom yes) (on_board yes) (fields_autoplaced)
+    (property "Reference" "#PWR0126" (id 0) (at 146.05 39.37 0)
+      (effects (font (size 1.27 1.27)) hide)
+    )
+    (property "Value" "GND" (id 1) (at 146.05 38.1 0))
+    (property "Footprint" "" (id 2) (at 146.05 33.02 0)
+      (effects (font (size 1.27 1.27)) hide)
+    )
+    (property "Datasheet" "" (id 3) (at 146.05 33.02 0)
+      (effects (font (size 1.27 1.27)) hide)
+    )
+    (pin "1")
+  )
   (symbol (lib_id "Device:LED") (at 52.07 161.29 90) (unit 1)
     (in_bom yes) (on_board yes)
-    (property "Reference" "LED" (id 0) (at 55.88 161.6074 90)
+    (property "Reference" "LED3" (id 0) (at 55.88 161.6074 90)
       (effects (font (size 1.27 1.27)) (justify right))
     )
@@
   (symbol (lib_id "Device:LED") (at 63.5 161.29 90) (unit 1)
     (in_bom yes) (on_board yes) (fields_autoplaced)
-    (property "Reference" "LED" (id 0) (at 67.31 161.6074 90)
+    (property "Reference" "LED4" (id 0) (at 67.31 161.6074 90)
       (effects (font (size 1.27 1.27)) (justify right))
     )
@@
   (symbol (lib_id "AE-BNO055:AE-BNO055") (at 50.8 77.47 0) (unit 1)
     (in_bom yes) (on_board yes) (fields_autoplaced)
-    (property "Reference" "AE-BNO055" (id 0) (at 56.515 72.39 0))
+    (property "Reference" "AE-BNO55" (id 0) (at 56.515 72.39 0))
     (property "Value" "AE-BNO055" (id 1) (at 56.515 74.93 0))
     (property "Footprint" "AE-BNO055:AE-BNO055" (id 2) (at 48.26 76.2 0)
@@
     (pin "9")
   )
+  (symbol (lib_id "Device:C_Polarized") (at 146.05 29.21 0) (unit 1)
+    (in_bom yes) (on_board yes) (fields_autoplaced)
+    (property "Reference" "C1" (id 0) (at 149.86 27.0509 0)
+      (effects (font (size 1.27 1.27)) (justify left))
+    )
+    (property "Value" "C_5V" (id 1) (at 149.86 29.5909 0)
+      (effects (font (size 1.27 1.27)) (justify left))
+    )
+    (property "Footprint" "Capacitor_THT:CP_Radial_D5.0mm_P2.50mm" (id 2) (at 147.0152 33.02 0)
+      (effects (font (size 1.27 1.27)) hide)
+    )
+    (property "Datasheet" "~" (id 3) (at 146.05 29.21 0)
+      (effects (font (size 1.27 1.27)) hide)
+    )
+    (pin "1")
+    (pin "2")
+  )
   (symbol (lib_id "Device:LED") (at 29.21 161.29 90) (unit 1)
     (in_bom yes) (on_board yes)
-    (property "Reference" "LED" (id 0) (at 33.02 161.6074 90)
+    (property "Reference" "LED1" (id 0) (at 33.02 161.6074 90)
       (effects (font (size 1.27 1.27)) (justify right))
     )
@@
   (symbol (lib_id "Device:LED") (at 88.9 161.29 90) (unit 1)
     (in_bom yes) (on_board yes) (fields_autoplaced)
-    (property "Reference" "LED" (id 0) (at 92.71 161.6074 90)
+    (property "Reference" "LED6" (id 0) (at 92.71 161.6074 90)
       (effects (font (size 1.27 1.27)) (justify right))
     )
@@
       (reference "#PWR0125") (unit 1) (value "+3.3V") (footprint "")
     )
+    (path "/ae7aeb91-d3e5-496e-a497-09d90e5fdde4"
+      (reference "#PWR0126") (unit 1) (value "GND") (footprint "")
+    )
+    (path "/49ec93f5-132d-48b0-b559-9a0a78ca6067"
+      (reference "#PWR0127") (unit 1) (value "+5V") (footprint "")
+    )
     (path "/d000c252-ded3-41d5-b3e4-49cb65069666"
-      (reference "AE-BNO055") (unit 1) (value "AE-BNO055") (footprint "AE-BNO055:AE-BNO055")
+      (reference "AE-BNO55") (unit 1) (value "AE-BNO055") (footprint "AE-BNO055:AE-BNO055")
     )
     (path "/e5435c51-2c5d-4ddb-9b5b-d7beb7cc7dac"
@@
       (reference "Air-UART1") (unit 1) (value "Air-UART") (footprint "Connector_JST:JST_XH_S4B-XH-A_1x04_P2.50mm_Horizontal")
     )
+    (path "/e8132e0a-e8b0-4762-bc9a-d87a76badf7a"
+      (reference "C1") (unit 1) (value "C_5V") (footprint "Capacitor_THT:CP_Radial_D5.0mm_P2.50mm")
+    )
     (path "/729b01ec-738f-43c5-822b-27d350075413"
       (reference "DPS310") (unit 1) (value "DPS310") (footprint "DPS310:DPS310")
@@
       (reference "J8") (unit 1) (value "Conn_01x03") (footprint "Connector_PinSocket_2.54mm:PinSocket_1x03_P2.54mm_Vertical")
     )
+    (path "/e8fe42a8-ca43-40a0-808f-01a629a50f73"
+      (reference "LED1") (unit 1) (value "SD") (footprint "LED_THT:LED_D3.0mm_Clear")
+    )
+    (path "/40dc120f-8d94-48d8-afb4-92f0e8601a29"
+      (reference "LED2") (unit 1) (value "ICS") (footprint "LED_THT:LED_D3.0mm_Clear")
+    )
+    (path "/b0cf4776-0395-4863-86c7-b7801a1cac53"
+      (reference "LED3") (unit 1) (value "Air") (footprint "LED_THT:LED_D3.0mm_Clear")
+    )
+    (path "/ca4f06d4-e667-4d24-afc1-294ab6c4ef73"
+      (reference "LED4") (unit 1) (value "Under") (footprint "LED_THT:LED_D3.0mm_Clear")
+    )
     (path "/18fb8f6b-b9c7-4385-ba05-b65cf395b9ea"
-      (reference "LED") (unit 1) (value "Power") (footprint "LED_THT:LED_D3.0mm_Clear")
-    )
-    (path "/40dc120f-8d94-48d8-afb4-92f0e8601a29"
-      (reference "LED") (unit 1) (value "ICS") (footprint "LED_THT:LED_D3.0mm_Clear")
-    )
-    (path "/b0cf4776-0395-4863-86c7-b7801a1cac53"
-      (reference "LED") (unit 1) (value "Air") (footprint "LED_THT:LED_D3.0mm_Clear")
-    )
-    (path "/ca4f06d4-e667-4d24-afc1-294ab6c4ef73"
-      (reference "LED") (unit 1) (value "Under") (footprint "LED_THT:LED_D3.0mm_Clear")
-    )
-    (path "/e8fe42a8-ca43-40a0-808f-01a629a50f73"
-      (reference "LED") (unit 1) (value "SD") (footprint "LED_THT:LED_D3.0mm_Clear")
+      (reference "LED5") (unit 1) (value "Power") (footprint "LED_THT:LED_D3.0mm_Clear")
     )
     (path "/edbca3e4-fedc-4bbf-9139-3f1d974c7d83"
-      (reference "LED") (unit 1) (value "1PPS") (footprint "LED_THT:LED_D3.0mm_Clear")
+      (reference "LED6") (unit 1) (value "1PPS") (footprint "LED_THT:LED_D3.0mm_Clear")
     )
     (path "/2fb9aea4-6f16-4bbe-8658-1d9caff83ec7"

Commit message: update
Parts:
- removed J7, J8: Conn_01x03, Connector_PinSocket_2.54mm:PinSocket_1x03_P2.54mm_Vertical, symbol Connector_Generic:Conn_01x03
- removed LED1: SD, LED_THT:LED_D3.0mm_Clear, symbol Device:LED
- removed LED2: ICS, LED_THT:LED_D3.0mm_Clear, symbol Device:LED
- removed LED3: Air, LED_THT:LED_D3.0mm_Clear, symbol Device:LED
- removed LED4: Under, LED_THT:LED_D3.0mm_Clear, symbol Device:LED
- removed LED5: Power, LED_THT:LED_D3.0mm_Clear, symbol Device:LED
- removed LED6: 1PPS, LED_THT:LED_D3.0mm_Clear, symbol Device:LED
- added LED1, LED2: Conn_01x04_Female, Connector_JST:JST_XH_S4B-XH-A_1x04_P2.50mm_Horizontal, symbol Connector:Conn_01x04_Female
- added U1: MOUDLE-SEEEDUINO-XIAO, XIAO_PCB:MOUDLE14P-2.54-21X17.8MM, symbol MOUDLE-SEEEDUINO-XIAO:MOUDLE-SEEEDUINO-XIAO
- GPS-UART1: value GPS-UART -> GPS-TWE-UART
Connections:
- net A12 is gone; now on net L_Under: J5.5 (Pin_5)
- net A13 is gone; now on net L_ICS: J5.6 (Pin_6)
- net TX0/1 is gone; now on net DTAR: J4.7 (Pin_7)
- net +3.3V: now also LED2.4 (Pin_4); no longer AE-MICRO-SD-DIP1.4 (VDD)
- net +5V: now also U1.14 (5V)
- net 1PPS: now also LED2.3 (Pin_3)
- net DRAT: now also J4.8 (Pin_8); no longer J6.4 (Pin_4)
- net DRUT: now also J6.4 (Pin_4); no longer J6.2 (Pin_2)
- net DTAR: no longer J6.3 (Pin_3)
- net DTUR: now also J6.3 (Pin_3); no longer J6.1 (Pin_1)
- net GND: now also LED1.1 (Pin_1), LED2.1 (Pin_1), U1.13 (GND)
- net IRXT: now also J6.2 (Pin_2); no longer J4.8 (Pin_8)
- net L_Air: now also J5.4 (Pin_4), LED1.4 (Pin_4); no longer J3.1 (Pin_1)
- net L_ICS: now also LED1.2 (Pin_2); no longer J2.5 (Pin_5)
- net L_SD: no longer J5.4 (Pin_4)
- net L_Under: now also LED1.3 (Pin_3); no longer J2.6 (Pin_6)
- net SD-CLK: now also U1.9 (PA7_A8_D8_SCK)
- net SD-CS: now also U1.1 (PA02_A0_D0); no longer J5.1 (Pin_1)
- net SD-MISO: now also U1.10 (PA5_A9_D9_MISO)
- net SD-MOSI: now also U1.11 (PA6_A10_D10_MOSI)
- net at ATP3012.15 (AOUT): no longer Speaker1.3 (Pin_3)
- new net *12: J2.6 (Pin_6)
- new net *13: J2.5 (Pin_5)
- new net A0: J3.1 (Pin_1)
- new net A8: J5.1 (Pin_1)
- new net DTSR: J6.1 (Pin_1), U1.8 (PB09_A7_D7_RX)
- new net RP3.3V: AE-MICRO-SD-DIP1.4 (VDD), U1.12 (3V3)
- no-connect marks 27 -> 24
Other:
- note added: "届かないので違法建築"
- moved on the sheet: AE-BNO55, DPS310

Commit message: update
Parts:
- added D1: D, Diode_THT:D_A-405_P12.70mm_Horizontal, symbol Device:D
- added D2, D3, D4: D, Diode_THT:D_A-405_P10.16mm_Horizontal, symbol Device:D
- added ICS-SW1: SW_DPDT_x2, Connector_PinHeader_2.54mm:PinHeader_1x03_P2.54mm_Vertical, symbol Switch:SW_DPDT_x2
- added Serial-SW1: SW_DPDT_x2, Button_Switch_THT:SW_Push_2P2T_Toggle_CK_PVA2OAH5xxxxxxV2, symbol Switch:SW_DPDT_x2
- U1: value MOUDLE-SEEEDUINO-XIAO -> SEEEDUINO-XIAO
Connections:
- net +5V: now also D1.2 (A); no longer U1.14 (5V)
- net DRAT: now also Serial-SW1.4 (A); no longer J4.8 (Pin_8)
- net DTAR: now also Serial-SW1.1 (A); no longer J4.7 (Pin_7)
- net IRXT: now also ICS-SW1.1 (A); no longer J6.2 (Pin_2)
- net VCC: now also D2.2 (A), D3.2 (A), D4.2 (A); no longer M78AR05-1.1 (IN), M78AR05-2.1 (IN), M78AR05-3.1 (IN)
- new net: D2.1 (K), M78AR05-1.1 (IN)
- new net: D4.1 (K), M78AR05-2.1 (IN)
- new net: D3.1 (K), M78AR05-3.1 (IN)
- new net: D1.1 (K), U1.14 (5V)
- new net RX0/0: J4.8 (Pin_8), Serial-SW1.5 (B)
- new net RX3/15: ICS-SW1.2 (B), J6.2 (Pin_2)
- new net TX0/1: J4.7 (Pin_7), Serial-SW1.2 (B)

Commit message: jlcpcb
Connections:
- net L_SD: now also LED2.2 (Pin_2), U1.2 (PA4_A1_D1)
- net at ATP3012.15 (AOUT): now also Speaker1.3 (Pin_3)
Other:
- note removed: "届かないので違法建築"
Changed lines of the file:
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@@
+    (stroke (width 0) (type default) (color 0 0 0 0))
+  )
+  (wire (pts (xy 246.38 58.42) (xy 255.27 58.42))
     (stroke (width 0) (type default) (color 0 0 0 0))
   )
@@
     (stroke (width 0) (type solid) (color 0 0 0 0))
   )
-  (text "届かないので違法建築" (at 246.38 62.23 0)
-    (effects (font (size 1.27 1.27)) (justify left bottom))
-  )
-  (text "届かないので違法建築" (at 59.69 186.69 0)
-    (effects (font (size 1.27 1.27)) (justify left bottom))
-  )
   (label "A10" (at 113.03 111.76 0)
     (effects (font (size 1.27 1.27)) (justify left bottom))
@@
     )
   )
-  (global_label "L_SD" (shape input) (at 29.21 83.82 180) (fields_autoplaced)
-    (effects (font (size 1.27 1.27)) (justify right))
-    (property "Intersheet References" "${INTERSHEET_REFS}" (id 0) (at 22.3217 83.8994 0)
+  (global_label "L_SD" (shape input) (at 31.75 83.82 180) (fields_autoplaced)
+    (effects (font (size 1.27 1.27)) (justify right))
+    (property "Intersheet References" "${INTERSHEET_REFS}" (id 0) (at 24.8617 83.8994 0)
       (effects (font (size 1.27 1.27)) (justify right) hide)
     )
@@
     )
   )
-  (global_label "L_SD" (shape input) (at 74.93 177.8 270) (fields_autoplaced)
-    (effects (font (size 1.27 1.27)) (justify right))
-    (property "Intersheet References" "${INTERSHEET_REFS}" (id 0) (at 75.0094 184.6883 90)
-      (effects (font (size 1.27 1.27)) (justify right) hide)
-    )
+  (global_label "L_SD" (shape input) (at 74.93 175.26 270) (fields_autoplaced)
+    (effects (font (size 1.27 1.27)) (justify right))
+    (property "Intersheet References" "${INTERSHEET_REFS}" (id 0) (at 75.0094 182.1483 90)
+      (effects (font (size 1.27 1.27)) (justify right) hide)
+    )
